File: PLC 32 V2.kicad_pcb (KiCad board)
At the start: 2 copper layers, 122.9 x 134.2 mm, 117 parts, among them J1 USB_C_Receptacle_USB2.0, J2 Screw_Terminal_01x05, J3 Screw_Terminal_01x05, J4 Screw_Terminal_01x02, J5 Screw_Terminal_01x10, J6 Screw_Terminal_01x02, J7 MODULO RTC, J8 Screw_Terminal_01x02, Q1 PMBT3904YS, Q2 FQP27P06, Q3 FQP27P06, Q4 FQP27P06, Q5 FQP27P06, Q6 FQP27P06, Q7 FQP27P06, Q8 BTA16-600C, Q9 BTA16-600C, SW1 SW_Push, SW2 SW_Push, U1 ILD74, U10 74HC14, U11 74HC14, U12 74HC14, U13 74HC14, U14 74HC14, U15 74HC14, U16 CH340C, U17 LM2576HVS-3.3, U18 ESP32-WROOM-32D, U2 ILD74, U21 ILD74, U22 ILD74, U23 ILD74, U24 ILD74, U25 ILD74, U26 ILD74, U27 MOC3021M, U28 MOC3021M, U29 ILD74, U3 ILD74, U30 74HC373, U4 ILD74, U5 ILD74, U6 ILD74, U7 ILD74, U8 74HC14, U9 74HC14

Commit message: add salidas separadas 1,2,3
Parts:
- removed C10: 470, Capacitor_SMD:C_Elec_10x10.2
- removed C11: 220, Capacitor_SMD:C_Elec_6.3x7.7
- removed C12, C13: 100n, Capacitor_THT:C_Rect_L31.5mm_W13.0mm_P27.50mm_MKS4
- removed C9: 100nF, Capacitor_SMD:C_0402_1005Metric
- removed J6, J8: Screw_Terminal_01x02, TerminalBlock:TerminalBlock_bornier-2_P5.08mm
- removed J7: MODULO RTC, Connector_PinHeader_2.54mm:PinHeader_1x04_P2.54mm_Vertical
- removed Q8, Q9: BTA16-600C, Package_TO_SOT_THT:TO-220-3_Vertical
- removed R41, R42: 330, Resistor_SMD:R_0603_1608Metric_Pad0.98x0.95mm_HandSolder
- removed R43, R46, R47: 220 ohm, Resistor_SMD:R_0603_1608Metric_Pad0.98x0.95mm_HandSolder
- removed R44, R45: 470, Resistor_THT:R_Axial_DIN0414_L11.9mm_D4.5mm_P15.24mm_Horizontal
- removed R48, R49: 330, Resistor_THT:R_Axial_DIN0207_L6.3mm_D2.5mm_P7.62mm_Horizontal
- removed R50, R51: 49, Resistor_THT:R_Axial_DIN0414_L11.9mm_D4.5mm_P15.24mm_Horizontal
- removed R52: 220 ohm, Resistor_SMD:R_0612_1632Metric
- removed U11, U12, U13, U14, U15: 74HC14, Package_SO:TSSOP-14_4.4x5mm_P0.65mm
- removed U16: CH340C, Package_SO:SOIC-16_3.9x9.9mm_P1.27mm
- removed U17: LM2576HVS-3.3, Package_TO_SOT_SMD:TO-263-5_TabPin3
- removed U18: ESP32-WROOM-32D, RF_Module:ESP32-WROOM-32
- removed U21, U22, U23, U24, U25, U26, U29: ILD74, Package_DIP:DIP-4_W7.62mm
- removed U27, U28: MOC3021M, Package_DIP:DIP-6_W7.62mm
- removed U30: 74HC373, Package_SO:SSOP-20_4.4x6.5mm_P0.65mm
- C7: value 100nF -> 470; footprint Capacitor_SMD:C_0402_1005Metric -> Capacitor_SMD:C_Elec_10x10.2
- C8: value 100nF -> 220; footprint Capacitor_SMD:C_0402_1005Metric -> Capacitor_SMD:C_Elec_6.3x7.7
- F1: value Fuse_Small -> Fuse
- J1: value USB_C_Receptacle_USB2.0 -> MODULO RTC; footprint Connector_USB:USB_C_Receptacle_HRO_TYPE-C-31-M-12 -> Connector_PinHeader_2.54mm:PinHeader_1x04_P2.54mm_Vertical
- J2: value Screw_Terminal_01x05 -> Salidas Q1 - Q5; footprint TerminalBlock:TerminalBlock_bornier-5_P5.08mm -> TerminalBlock_Phoenix:TerminalBlock_Phoenix_PT-1,5-10-5.0-H_1x10_P5.00mm_Horizontal
- J3: value Screw_Terminal_01x05 -> Input_1
- J4: value Screw_Terminal_01x02 -> Input_2; footprint TerminalBlock:TerminalBlock_bornier-2_P5.08mm -> TerminalBlock:TerminalBlock_bornier-5_P5.08mm
- J5: value Screw_Terminal_01x10 -> DC_IN; footprint TerminalBlock_Phoenix:TerminalBlock_Phoenix_PT-1,5-10-5.0-H_1x10_P5.00mm_Horizontal -> TerminalBlock:TerminalBlock_bornier-2_P5.08mm
- L1: moved to F.Cu
- Q1: value PMBT3904YS -> FQP27P06; footprint Package_TO_SOT_SMD:SOT-363_SC-70-6 -> Package_TO_SOT_SMD:TO-252-3_TabPin2
- Q2, Q3, Q4, Q5, Q6: footprint Package_TO_SOT_SMD:TO-252-2_TabPin1 -> Package_TO_SOT_SMD:TO-252-3_TabPin2
- Q7: value FQP27P06 -> PMBT3904YS; footprint Package_TO_SOT_SMD:TO-252-2_TabPin1 -> Package_TO_SOT_SMD:SOT-363_SC-70-6
- R1, R2, R3: value 20k -> 10k; footprint Resistor_SMD:R_0603_1608Metric_Pad0.98x0.95mm_HandSolder -> Resistor_SMD:R_0603_1608Metric
- R10, R11, R13, R14, R9: value 1k -> 220 ohm; footprint Resistor_SMD:R_0603_1608Metric_Pad0.98x0.95mm_HandSolder -> Resistor_SMD:R_0603_1608Metric
- R12, R15, R19: value 10k -> 220 ohm; footprint Resistor_SMD:R_0603_1608Metric_Pad0.98x0.95mm_HandSolder -> Resistor_SMD:R_0603_1608Metric
- R16, R17, R18, R20, R21, R22, R23, R24, R25, R26, R27, R28, R29, R30: footprint Resistor_SMD:R_0603_1608Metric_Pad0.98x0.95mm_HandSolder -> Resistor_SMD:R_0603_1608Metric
- R31, R32, R33, R34, R35, R36: value 220 ohm -> 20k; footprint Resistor_SMD:R_0603_1608Metric_Pad0.98x0.95mm_HandSolder -> Resistor_SMD:R_0603_1608Metric
- R37: value 220 ohm -> 1k; footprint Resistor_SMD:R_0603_1608Metric_Pad0.98x0.95mm_HandSolder -> Resistor_SMD:R_0603_1608Metric
- R38: value 220 ohm -> 10k; footprint Resistor_SMD:R_0603_1608Metric_Pad0.98x0.95mm_HandSolder -> Resistor_SMD:R_0603_1608Metric
- R39: value 220 ohm -> 1k
- R4, R5, R7, R8: value 20k -> 220 ohm; footprint Resistor_SMD:R_0603_1608Metric_Pad0.98x0.95mm_HandSolder -> Resistor_SMD:R_0603_1608Metric
- R40: value 10k -> 1k; footprint Resistor_SMD:R_0603_1608Metric_Pad0.98x0.95mm_HandSolder -> Resistor_SMD:R_0603_1608Metric
- R6: value 20k -> 220 ohm
- SW1: value SW_Push -> RST
- SW2: value SW_Push -> PRG
- U1, U2, U3, U4, U5, U7: value ILD74 -> LD74-X009T; footprint Package_DIP:DIP-4_W7.62mm -> Package_DIP:DIP-8_W8.89mm_SMDSocket_LongPads
- U10: value 74HC14 -> ESP32-WROOM-32D; footprint Package_SO:TSSOP-14_4.4x5mm_P0.65mm -> RF_Module:ESP32-WROOM-32
- U6: value ILD74 -> 74HC14; footprint Package_DIP:DIP-4_W7.62mm -> Package_SO:SOIC-14W_7.5x9mm_P1.27mm
- U8: value 74HC14 -> 74HC373; footprint Package_SO:TSSOP-14_4.4x5mm_P0.65mm -> Package_SO:SSOP-20_4.4x6.5mm_P0.65mm
- U9: value 74HC14 -> LM2576HVS-3.3; footprint Package_SO:TSSOP-14_4.4x5mm_P0.65mm -> Package_TO_SOT_SMD:TO-263-5_TabPin3
- moved R10 243.0 mm to (117.3, 89.1)
- moved R9 240.0 mm to (141.7, 62.7)
- moved R14 232.5 mm to (138.3, 60.2)
- moved R30 221.9 mm to (109.3, 84.1)
- moved R29 216.6 mm to (127.5, 75.5)
- moved R32 211.7 mm to (163.9, 119.7)
- moved R18 205.0 mm to (146.3, 57.7)
- moved R17 195.4 mm to (117.3, 84.1)
- moved R19 194.2 mm to (137.7, 68.7)
- moved R24 188.9 mm to (113.3, 89.1)
- moved R22 185.5 mm to (142.3, 57.7)
- moved R23 182.5 mm to (138.3, 57.7)
- moved R31 180.3 mm to (173.5, 118.4)
- moved R33 174.5 mm to (159.9, 119.7)
- moved D1 172.9 mm to (95.4, 115.8)
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Connections:
- C8 pad 1: Net-(C8-Pad1) -> VCC
- D2 pad 1: Net-(C10-Pad1) -> Net-(C7-Pad1)
- J2 pad 1: IN01 -> 3L
- J2 pad 2: IN02 -> M3
- J2 pad 3: IN03 -> Q1
- J2 pad 4: IN04 -> Q2
- J2 pad 5: Net-(D1-Pad2) -> Q3
- J3 pad 1: Net-(D1-Pad2) -> IN01
- J3 pad 2: IA08 -> IN02
- J3 pad 3: IA07 -> IN03
- J3 pad 4: IN06 -> IN04
- J3 pad 5: IN05 -> Net-(D1-Pad2)
- J4 pad 1: GND -> Net-(D1-Pad2)
- J4 pad 2: Net-(F1-Pad1) -> IA08
- J5 pad 1: 3L -> Net-(F1-Pad1)
- J5 pad 2: M3 -> GND
- Q1 pad 1: DTR -> Net-(Q1-Pad1)
- Q1 pad 2: Net-(Q1-Pad2) -> 3L
- Q1 pad 3: RTS -> Q1
- Q2 pad 2: Q1 -> 3L
- Q3 pad 2: Q2 -> 3L
- Q4 pad 1: Net-(Q4-Pad1) -> Net-(R22-Pad2)
- Q4 pad 2: Q3 -> 2L
- Q5 pad 1: Net-(Q5-Pad1) -> Net-(R24-Pad2)
- Q5 pad 2: Q4 -> 2L
- Q6 pad 1: Net-(Q6-Pad1) -> Net-(R26-Pad2)
- Q6 pad 2: Q5 -> 2L
- Q7 pad 1: Net-(Q7-Pad1) -> /BTN_RST_PRG/DTR
- Q7 pad 2: Q6 -> Net-(R40-Pad2)
- R1 pad 1: IN01 -> IO2
- R1 pad 2: Net-(R1-Pad2) -> GND
- R10 pad 1: Net-(R10-Pad1) -> M3
- R10 pad 2: Tx -> Q2
- R11 pad 1: VCC -> Net-(R11-Pad1)
- R11 pad 2: IO0 -> Net-(Q3-Pad1)
- R12 pad 1: EN -> M3
- R12 pad 2: VCC -> Q3
- R13 pad 1: DTR -> Net-(R13-Pad1)
- R13 pad 2: Net-(Q1-Pad5) -> 3L
- R14 pad 1: RTS -> Net-(R14-Pad1)
- R14 pad 2: Net-(Q1-Pad2) -> 3L
- R15 pad 1: IO2 -> Net-(R11-Pad1)
- R15 pad 2: GND -> 3L
- R16 pad 1: IO4 -> IO12
- R17 pad 1: IO5 -> IO14
- R18 pad 1: IO12 -> IO13
- R19 pad 1: IO13 -> IO12
- R19 pad 2: GND -> Net-(R19-Pad2)
- R2 pad 1: IN02 -> IO4
- R2 pad 2: Net-(R2-Pad2) -> GND
- R20 pad 1: IO2 -> IO14
- R21 pad 1: IO4 -> IO13
- R22 pad 1: IO5 -> Net-(R22-Pad1)
- R23 pad 1: IO12 -> M3
- R23 pad 2: Net-(R23-Pad2) -> Q4
- R24 pad 1: IO13 -> Net-(R24-Pad1)
- R25 pad 1: Net-(R25-Pad1) -> M3
- R25 pad 2: Net-(Q2-Pad1) -> Q5
- R26 pad 1: M3 -> Net-(R26-Pad1)
- R26 pad 2: Q1 -> Net-(R26-Pad2)
- R27 pad 1: Net-(R27-Pad1) -> M3
- R27 pad 2: Net-(Q3-Pad1) -> Q6
- R28 pad 1: M3 -> Net-(R22-Pad1)
- R28 pad 2: Q2 -> 2L
- R29 pad 1: Net-(R29-Pad1) -> Net-(R24-Pad1)
- R29 pad 2: Net-(Q4-Pad1) -> 2L
- R3 pad 1: IN03 -> IO5
- R3 pad 2: Net-(R3-Pad2) -> GND
- R30 pad 1: M3 -> Net-(R26-Pad1)
- R30 pad 2: Q3 -> 2L
- R31 pad 1: Net-(R31-Pad1) -> IN01
- R31 pad 2: Net-(Q5-Pad1) -> Net-(R31-Pad2)
- R32 pad 1: M3 -> IN02
- R32 pad 2: Q4 -> Net-(R32-Pad2)
- R33 pad 1: Net-(R33-Pad1) -> IN04
- R33 pad 2: Net-(Q6-Pad1) -> Net-(R33-Pad2)
- R34 pad 1: M3 -> IN03
- R34 pad 2: Q5 -> Net-(R34-Pad2)
- R35 pad 1: Net-(R25-Pad1) -> IN05
- R35 pad 2: 3L -> Net-(R35-Pad2)
- R36 pad 1: Net-(R27-Pad1) -> IN06
- R36 pad 2: 3L -> Net-(R36-Pad2)
- R37 pad 1: Net-(R29-Pad1) -> VCC
- R37 pad 2: 3L -> IO0
- R38 pad 1: Net-(R31-Pad1) -> EN
- R38 pad 2: 3L -> VCC
- R39 pad 1: Net-(R33-Pad1) -> /BTN_RST_PRG/DTR
- R39 pad 2: 2L -> Net-(R39-Pad2)
- R4 pad 1: IN04 -> IO2
- R40 pad 1: IO14 -> /BTN_RST_PRG/RTS
- R40 pad 2: GND -> Net-(R40-Pad2)
- R5 pad 1: IN05 -> IO4
- R6 pad 1: IN06 -> IO5
- R7 pad 1: IA07 -> Net-(R13-Pad1)
- R7 pad 2: Net-(R7-Pad2) -> Net-(Q1-Pad1)
- R8 pad 1: IA08 -> M3
- R8 pad 2: Net-(R8-Pad2) -> Q1
- R9 pad 1: Net-(R9-Pad1) -> Net-(R14-Pad1)
- R9 pad 2: Rx -> Net-(Q2-Pad1)
- U1 pad 1: Net-(R1-Pad2) -> Net-(R4-Pad2)
- U1 pad 2: IN -> GND
- U1 pad 3: (no net) -> GND
- U1 pad 4: (no net) -> Net-(R5-Pad2)
- U10 pad 1: (no net) -> GND
- U10 pad 10: (no net) -> IO25
- U10 pad 11: (no net) -> IO26
- U10 pad 12: (no net) -> IO27
- U10 pad 13: (no net) -> IO14
- U10 pad 14: (no net) -> IO12
- U10 pad 2: (no net) -> VCC
- U10 pad 3: Net-(C3-Pad1) -> EN
- U10 pad 4: D_3 -> IO36
- U10 pad 5: (no net) -> unconnected-(U10-Pad5)
- U10 pad 6: (no net) -> IO34
- U10 pad 7: (no net) -> IO35
- U10 pad 8: (no net) -> IO32
- U10 pad 9: (no net) -> IO33
- U2 pad 1: (no net) -> Net-(R6-Pad2)
- U2 pad 2: (no net) -> GND
- U2 pad 3: IN -> GND
- U2 pad 4: Net-(R3-Pad2) -> Net-(R19-Pad2)
- U3 pad 1: (no net) -> Net-(R20-Pad2)
- U3 pad 2: (no net) -> GND
- U3 pad 3: IN -> GND
- U3 pad 4: Net-(R4-Pad2) -> Net-(R21-Pad2)
- U4 pad 1: (no net) -> Net-(R31-Pad2)
- U4 pad 2: (no net) -> IN
- U4 pad 4: Net-(R5-Pad2) -> Net-(R32-Pad2)
- U5 pad 1: (no net) -> Net-(R33-Pad2)
- U5 pad 2: (no net) -> IN
- U5 pad 4: Net-(R6-Pad2) -> Net-(R34-Pad2)
- U6 pad 1: (no net) -> Net-(C1-Pad1)
- U6 pad 2: (no net) -> D_1
- U6 pad 3: IN -> Net-(C2-Pad1)
- U6 pad 4: Net-(R7-Pad2) -> D_2
- U7 pad 1: (no net) -> Net-(R35-Pad2)
- U7 pad 2: (no net) -> IN
- U7 pad 4: Net-(R8-Pad2) -> Net-(R36-Pad2)
- U8 pad 1: (no net) -> GND
- U8 pad 10: (no net) -> GND
- U8 pad 11: (no net) -> GND
- U8 pad 12: (no net) -> IO32
- U8 pad 13: (no net) -> D_5
- U8 pad 14: (no net) -> D_6
- U8 pad 2: (no net) -> IO17
- U8 pad 3: Net-(C1-Pad1) -> D_1
- U8 pad 4: D_1 -> D_2
- U8 pad 5: (no net) -> IO18
- U8 pad 6: (no net) -> IO19
- U8 pad 7: (no net) -> D_3
- U8 pad 8: (no net) -> D_4
- U8 pad 9: (no net) -> IO23
- U9 pad 1: (no net) -> Net-(C7-Pad1)
- U9 pad 2: (no net) -> Net-(D3-Pad1)
- U9 pad 3: Net-(C2-Pad1) -> GND
- U9 pad 4: D_2 -> VCC
- U9 pad 5: (no net) -> GND
Routing:
- net 2L: track 125.3 -> 0.00 mm
- net GND: track 67.2 -> 0.00 mm
- net Net-(Q9-Pad3): track 16.6 -> 0.00 mm
- net Net-(C12-Pad1): track 16.1 -> 0.00 mm
- net Net-(Q8-Pad3): track 15.3 -> 0.00 mm
- net Net-(C13-Pad1): track 15.1 -> 0.00 mm
Other:
- board outline removed

Commit message: add entradas separadas
Parts:
- removed C1, C2, C3, C4, C5, C6: 100nF, Capacitor_SMD:C_0402_1005Metric
- removed C7: 470, Capacitor_SMD:C_Elec_10x10.2
- removed C8: 220, Capacitor_SMD:C_Elec_6.3x7.7
- removed D1, D2, D3: B330, Diode_SMD:D_0402_1005Metric
- removed F1: Fuse, Fuse:Fuse_0805_2012Metric
- removed J1: MODULO RTC, Connector_PinHeader_2.54mm:PinHeader_1x04_P2.54mm_Vertical
- removed J2: Salidas Q1 - Q5, TerminalBlock_Phoenix:TerminalBlock_Phoenix_PT-1,5-10-5.0-H_1x10_P5.00mm_Horizontal
- removed J3: Input_1, TerminalBlock:TerminalBlock_bornier-5_P5.08mm
- removed J4: Input_2, TerminalBlock:TerminalBlock_bornier-5_P5.08mm
- removed J5: DC_IN, TerminalBlock:TerminalBlock_bornier-2_P5.08mm
- removed L1: 100u, Inductor_SMD:L_TDK_SLF10165
- removed Q1, Q2, Q3, Q4, Q5, Q6: FQP27P06, Package_TO_SOT_SMD:TO-252-3_TabPin2
- removed Q7: PMBT3904YS, Package_TO_SOT_SMD:SOT-363_SC-70-6
- removed R1, R16, R17, R18, R2, R3, R38: 10k, Resistor_SMD:R_0603_1608Metric
- removed R10, R11, R12, R13, R14, R15, R19, R20, R21, R22, R23, R24, R25, R26, R27, R28, R29, R30, R4, R5, R7, R8, R9: 220 ohm, Resistor_SMD:R_0603_1608Metric
- removed R31, R32, R33, R34, R35, R36: 20k, Resistor_SMD:R_0603_1608Metric
- removed R37, R40: 1k, Resistor_SMD:R_0603_1608Metric
- removed R39: 1k, Resistor_SMD:R_0603_1608Metric_Pad0.98x0.95mm_HandSolder
- removed R6: 220 ohm, Resistor_SMD:R_0603_1608Metric_Pad0.98x0.95mm_HandSolder
- removed SW1: RST, Button_Switch_SMD:SW_SPST_CK_RS282G05A3
- removed SW2: PRG, Button_Switch_SMD:SW_SPST_CK_RS282G05A3
- removed U1, U2, U3, U4, U5, U7: LD74-X009T, Package_DIP:DIP-8_W8.89mm_SMDSocket_LongPads
- removed U10: ESP32-WROOM-32D, RF_Module:ESP32-WROOM-32
- removed U6: 74HC14, Package_SO:SOIC-14W_7.5x9mm_P1.27mm
- removed U8: 74HC373, Package_SO:SSOP-20_4.4x6.5mm_P0.65mm
- removed U9: LM2576HVS-3.3, Package_TO_SOT_SMD:TO-263-5_TabPin3
