File: btn_rst_prg.kicad_sch (KiCad schematic)
At the start: 7 parts, among them Q1 PMBT3904YS, SW1 RST, SW2 PRG

Commit message: add
Parts:
- R1: renamed from R4; value 1k -> 10k
- renumbered R1 to R2, R2 to R3, R3 to R4
Changed lines of the file:
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@@
   (junction (at 55.88 124.46) (diameter 0) (color 0 0 0 0)
   )
-  (junction (at 55.88 130.81) (diameter 0) (color 0 0 0 0)
-  )
   (junction (at 97.79 124.46) (diameter 0) (color 0 0 0 0)
   )
@@
     (stroke (width 0) (type default))
   )
-  (wire (pts (xy 50.8 130.81) (xy 55.88 130.81))
-    (stroke (width 0) (type default))
-  )
   (wire (pts (xy 90.17 135.89) (xy 90.17 140.97))
     (stroke (width 0) (type default))
@@
     (stroke (width 0) (type default))
   )
-  (wire (pts (xy 55.88 130.81) (xy 55.88 135.89))
+  (wire (pts (xy 55.88 124.46) (xy 55.88 135.89))
     (stroke (width 0) (type default))
   )
@@
   )
   (wire (pts (xy 110.49 113.03) (xy 135.89 113.03))
-    (stroke (width 0) (type default))
-  )
-  (wire (pts (xy 55.88 124.46) (xy 55.88 130.81))
     (stroke (width 0) (type default))
   )
@@
     (effects (font (size 5.08 5.08) (thickness 1.016) bold) (justify left bottom))
   )
-  (hierarchical_label "GND" (shape input) (at 50.8 130.81 180) (fields_autoplaced)
-    (effects (font (size 1.27 1.27)) (justify right))
-  )
   (hierarchical_label "VCC" (shape input) (at 96.52 87.63 0) (fields_autoplaced)
     (effects (font (size 1.27 1.27)) (justify left))
@@
   (symbol (lib_id "Device:R") (at 93.98 93.98 180) (unit 1)
     (in_bom yes) (on_board yes) (dnp no)
-    (property "Reference" "R1" (at 91.44 93.98 90)
+    (property "Reference" "R2" (at 91.44 93.98 90)
       (effects (font (size 1.27 1.27)))
     )
@@
       (project "PLC 32 V2"
         (path "/d17a54f1-6eda-453f-95e1-42a53b02a1c3/42521a84-9a19-4c46-b1f2-db09ca0e83df"
-          (reference "R1") (unit 1) (value "10k") (footprint "Resistor_SMD:R_0603_1608Metric")
+          (reference "R2") (unit 1) (value "10k") (footprint "Resistor_SMD:R_0603_1608Metric")
         )
       )
@@
   (symbol (lib_id "Device:R") (at 128.27 104.14 270) (unit 1)
     (in_bom yes) (on_board yes) (dnp no)
-    (property "Reference" "R2" (at 128.27 106.68 90)
+    (property "Reference" "R3" (at 128.27 106.68 90)
       (effects (font (size 1.27 1.27)))
     )
@@
       (project "PLC 32 V2"
         (path "/d17a54f1-6eda-453f-95e1-42a53b02a1c3/42521a84-9a19-4c46-b1f2-db09ca0e83df"
-          (reference "R2") (unit 1) (value "1k") (footprint "Resistor_SMD:R_0603_1608Metric_Pad0.98x0.95mm_HandSolder")
+          (reference "R3") (unit 1) (value "1k") (footprint "Resistor_SMD:R_0603_1608Metric_Pad0.98x0.95mm_HandSolder")
         )
       )
@@
   (symbol (lib_id "Device:R") (at 128.27 124.46 270) (unit 1)
     (in_bom yes) (on_board yes) (dnp no)
-    (property "Reference" "R3" (at 128.27 127 90)
+    (property "Reference" "R4" (at 128.27 127 90)
       (effects (font (size 1.27 1.27)))
     )
@@
       (project "PLC 32 V2"
         (path "/d17a54f1-6eda-453f-95e1-42a53b02a1c3/42521a84-9a19-4c46-b1f2-db09ca0e83df"
-          (reference "R3") (unit 1) (value "1k") (footprint "Resistor_SMD:R_0603_1608Metric")
+          (reference "R4") (unit 1) (value "1k") (footprint "Resistor_SMD:R_0603_1608Metric")
         )
       )
@@
   (symbol (lib_id "Device:R") (at 90.17 132.08 180) (unit 1)
     (in_bom yes) (on_board yes) (dnp no)
-    (property "Reference" "R4" (at 87.63 132.08 90)
-      (effects (font (size 1.27 1.27)))
-    )
-    (property "Value" "1k" (at 90.17 132.08 90)
+    (property "Reference" "R1" (at 87.63 132.08 90)
+      (effects (font (size 1.27 1.27)))
+    )
+    (property "Value" "10k" (at 90.17 132.08 90)
       (effects (font (size 1.27 1.27)))
     )
@@
       (project "PLC 32 V2"
         (path "/d17a54f1-6eda-453f-95e1-42a53b02a1c3/42521a84-9a19-4c46-b1f2-db09ca0e83df"
-          (reference "R4") (unit 1) (value "1k") (footprint "Resistor_SMD:R_0603_1608Metric")
-        )
-      )
+          (reference "R1") (unit 1) (value "10k") (footprint "Resistor_SMD:R_0603_1608Metric")
+        )
+      )
