File: salida1.kicad_sch (KiCad schematic)
At the start: 7 parts, among them Q2 FQP27P06, U8 LD74-X009T

Commit message: add
Parts:
- renumbered R11 to R5, R12 to R6, R13 to R7, R14 to R8, R15 to R9, U8 to U4
Changed lines of the file:
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@@
   (symbol (lib_id "Device:R") (at 68.58 127 0) (unit 1)
     (in_bom yes) (on_board yes) (dnp no) (fields_autoplaced)
-    (property "Reference" "R11" (at 71.12 125.7299 0)
+    (property "Reference" "R5" (at 71.12 125.7299 0)
       (effects (font (size 1.27 1.27)) (justify left))
     )
@@
       (project "PLC 32 V2"
         (path "/d17a54f1-6eda-453f-95e1-42a53b02a1c3/ee71d592-407c-4f0c-90d3-cb4773606332"
-          (reference "R11") (unit 1) (value "10k") (footprint "Resistor_SMD:R_0603_1608Metric")
+          (reference "R5") (unit 1) (value "10k") (footprint "Resistor_SMD:R_0603_1608Metric")
         )
       )
@@
   (symbol (lib_id "Device:R") (at 120.65 128.27 90) (unit 1)
     (in_bom yes) (on_board yes) (dnp no)
-    (property "Reference" "R14" (at 118.11 130.81 90)
+    (property "Reference" "R8" (at 118.11 130.81 90)
       (effects (font (size 1.27 1.27)))
     )
@@
       (project "PLC 32 V2"
         (path "/d17a54f1-6eda-453f-95e1-42a53b02a1c3/ee71d592-407c-4f0c-90d3-cb4773606332"
-          (reference "R14") (unit 1) (value "220 ohm") (footprint "Resistor_SMD:R_0603_1608Metric")
+          (reference "R8") (unit 1) (value "220 ohm") (footprint "Resistor_SMD:R_0603_1608Metric")
         )
       )
@@
   (symbol (lib_id "Device:R") (at 78.74 119.38 90) (unit 1)
     (in_bom yes) (on_board yes) (dnp no) (fields_autoplaced)
-    (property "Reference" "R12" (at 78.74 113.03 90)
+    (property "Reference" "R6" (at 78.74 113.03 90)
       (effects (font (size 1.27 1.27)))
     )
@@
       (project "PLC 32 V2"
         (path "/d17a54f1-6eda-453f-95e1-42a53b02a1c3/ee71d592-407c-4f0c-90d3-cb4773606332"
-          (reference "R12") (unit 1) (value "220 ohm") (footprint "Resistor_SMD:R_0603_1608Metric")
+          (reference "R6") (unit 1) (value "220 ohm") (footprint "Resistor_SMD:R_0603_1608Metric")
         )
       )
@@
   (symbol (lib_id "Device:R") (at 120.65 119.38 90) (unit 1)
     (in_bom yes) (on_board yes) (dnp no)
-    (property "Reference" "R13" (at 115.57 118.11 90)
+    (property "Reference" "R7" (at 115.57 118.11 90)
       (effects (font (size 1.27 1.27)))
     )
@@
       (project "PLC 32 V2"
         (path "/d17a54f1-6eda-453f-95e1-42a53b02a1c3/ee71d592-407c-4f0c-90d3-cb4773606332"
-          (reference "R13") (unit 1) (value "220 ohm") (footprint "Resistor_SMD:R_0603_1608Metric")
+          (reference "R7") (unit 1) (value "220 ohm") (footprint "Resistor_SMD:R_0603_1608Metric")
         )
       )
@@
   (symbol (lib_id "Isolator:ILD74") (at 97.79 121.92 0) (unit 1)
     (in_bom yes) (on_board yes) (dnp no) (fields_autoplaced)
-    (property "Reference" "U8" (at 97.79 114.3 0)
+    (property "Reference" "U4" (at 97.79 114.3 0)
       (effects (font (size 1.27 1.27)))
     )
@@
       (project "PLC 32 V2"
         (path "/d17a54f1-6eda-453f-95e1-42a53b02a1c3/ee71d592-407c-4f0c-90d3-cb4773606332"
-          (reference "U8") (unit 1) (value "LD74-X009T") (footprint "Package_DIP:DIP-8_W8.89mm_SMDSocket_LongPads")
+          (reference "U4") (unit 1) (value "LD74-X009T") (footprint "Package_DIP:DIP-8_W8.89mm_SMDSocket_LongPads")
         )
       )
@@
   (symbol (lib_id "Device:R") (at 129.54 113.03 90) (unit 1)
     (in_bom yes) (on_board yes) (dnp no)
-    (property "Reference" "R15" (at 125.73 110.49 90)
+    (property "Reference" "R9" (at 125.73 110.49 90)
       (effects (font (size 1.27 1.27)))
     )
@@
       (project "PLC 32 V2"
         (path "/d17a54f1-6eda-453f-95e1-42a53b02a1c3/ee71d592-407c-4f0c-90d3-cb4773606332"
-          (reference "R15") (unit 1) (value "220 ohm") (footprint "Resistor_SMD:R_0603_1608Metric")
+          (reference "R9") (unit 1) (value "220 ohm") (footprint "Resistor_SMD:R_0603_1608Metric")
         )
       )
