File: salida2.kicad_sch (KiCad schematic)
At the start: 7 parts, among them Q3 FQP27P06, U8 LD74-X009T

Commit message: add
Parts:
- renumbered R16 to R10, R17 to R11, R18 to R12, R19 to R13, R20 to R14, U8 to U4
Changed lines of the file:
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@@
   (symbol (lib_id "Device:R") (at 120.65 130.81 90) (unit 1)
     (in_bom yes) (on_board yes) (dnp no)
-    (property "Reference" "R19" (at 118.11 133.35 90)
+    (property "Reference" "R13" (at 118.11 133.35 90)
       (effects (font (size 1.27 1.27)))
     )
@@
       (project "PLC 32 V2"
         (path "/d17a54f1-6eda-453f-95e1-42a53b02a1c3/2637b07c-4b5f-4e3d-b3e5-25bd73194631"
-          (reference "R19") (unit 1) (value "220 ohm") (footprint "Resistor_SMD:R_0603_1608Metric")
+          (reference "R13") (unit 1) (value "220 ohm") (footprint "Resistor_SMD:R_0603_1608Metric")
         )
       )
@@
   (symbol (lib_id "Device:R") (at 68.58 129.54 0) (unit 1)
     (in_bom yes) (on_board yes) (dnp no) (fields_autoplaced)
-    (property "Reference" "R16" (at 71.12 128.2699 0)
+    (property "Reference" "R10" (at 71.12 128.2699 0)
       (effects (font (size 1.27 1.27)) (justify left))
     )
@@
       (project "PLC 32 V2"
         (path "/d17a54f1-6eda-453f-95e1-42a53b02a1c3/2637b07c-4b5f-4e3d-b3e5-25bd73194631"
-          (reference "R16") (unit 1) (value "10k") (footprint "Resistor_SMD:R_0603_1608Metric")
+          (reference "R10") (unit 1) (value "10k") (footprint "Resistor_SMD:R_0603_1608Metric")
         )
       )
@@
   (symbol (lib_id "Device:R") (at 129.54 115.57 90) (unit 1)
     (in_bom yes) (on_board yes) (dnp no)
-    (property "Reference" "R20" (at 125.73 111.76 90)
+    (property "Reference" "R14" (at 125.73 111.76 90)
       (effects (font (size 1.27 1.27)))
     )
@@
       (project "PLC 32 V2"
         (path "/d17a54f1-6eda-453f-95e1-42a53b02a1c3/2637b07c-4b5f-4e3d-b3e5-25bd73194631"
-          (reference "R20") (unit 1) (value "220 ohm") (footprint "Resistor_SMD:R_0603_1608Metric")
+          (reference "R14") (unit 1) (value "220 ohm") (footprint "Resistor_SMD:R_0603_1608Metric")
         )
       )
@@
   (symbol (lib_id "Device:R") (at 78.74 121.92 90) (unit 1)
     (in_bom yes) (on_board yes) (dnp no) (fields_autoplaced)
-    (property "Reference" "R17" (at 78.74 115.57 90)
+    (property "Reference" "R11" (at 78.74 115.57 90)
       (effects (font (size 1.27 1.27)))
     )
@@
       (project "PLC 32 V2"
         (path "/d17a54f1-6eda-453f-95e1-42a53b02a1c3/2637b07c-4b5f-4e3d-b3e5-25bd73194631"
-          (reference "R17") (unit 1) (value "220 ohm") (footprint "Resistor_SMD:R_0603_1608Metric")
+          (reference "R11") (unit 1) (value "220 ohm") (footprint "Resistor_SMD:R_0603_1608Metric")
         )
       )
@@
   (symbol (lib_id "Isolator:ILD74") (at 97.79 124.46 0) (unit 2)
     (in_bom yes) (on_board yes) (dnp no) (fields_autoplaced)
-    (property "Reference" "U8" (at 97.79 116.84 0)
+    (property "Reference" "U4" (at 97.79 116.84 0)
       (effects (font (size 1.27 1.27)))
     )
@@
       (project "PLC 32 V2"
         (path "/d17a54f1-6eda-453f-95e1-42a53b02a1c3/2637b07c-4b5f-4e3d-b3e5-25bd73194631"
-          (reference "U8") (unit 2) (value "LD74-X009T") (footprint "Package_DIP:DIP-8_W8.89mm_SMDSocket_LongPads")
+          (reference "U4") (unit 2) (value "LD74-X009T") (footprint "Package_DIP:DIP-8_W8.89mm_SMDSocket_LongPads")
         )
       )
@@
   (symbol (lib_id "Device:R") (at 120.65 121.92 90) (unit 1)
     (in_bom yes) (on_board yes) (dnp no)
-    (property "Reference" "R18" (at 118.11 120.65 90)
+    (property "Reference" "R12" (at 118.11 120.65 90)
       (effects (font (size 1.27 1.27)))
     )
@@
       (project "PLC 32 V2"
         (path "/d17a54f1-6eda-453f-95e1-42a53b02a1c3/2637b07c-4b5f-4e3d-b3e5-25bd73194631"
-          (reference "R18") (unit 1) (value "220 ohm") (footprint "Resistor_SMD:R_0603_1608Metric")
+          (reference "R12") (unit 1) (value "220 ohm") (footprint "Resistor_SMD:R_0603_1608Metric")
         )
       )
