File: salida3.kicad_sch (KiCad schematic)
At the start: 7 parts, among them Q4 FQP27P06, U9 LD74-X009T

Commit message: add
Parts:
- renumbered R21 to R15, R22 to R16, R23 to R17, R24 to R18, R25 to R19, U9 to U5
Changed lines of the file:
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@@
   (symbol (lib_id "Device:R") (at 66.04 139.7 0) (unit 1)
     (in_bom yes) (on_board yes) (dnp no) (fields_autoplaced)
-    (property "Reference" "R21" (at 68.58 138.4299 0)
+    (property "Reference" "R15" (at 68.58 138.4299 0)
       (effects (font (size 1.27 1.27)) (justify left))
     )
@@
       (project "PLC 32 V2"
         (path "/d17a54f1-6eda-453f-95e1-42a53b02a1c3/e0987795-0f8d-4564-9094-c23cc01406e8"
-          (reference "R21") (unit 1) (value "10k") (footprint "Resistor_SMD:R_0603_1608Metric")
+          (reference "R15") (unit 1) (value "10k") (footprint "Resistor_SMD:R_0603_1608Metric")
         )
       )
@@
   (symbol (lib_id "Device:R") (at 127 125.73 90) (unit 1)
     (in_bom yes) (on_board yes) (dnp no)
-    (property "Reference" "R25" (at 123.19 121.92 90)
+    (property "Reference" "R19" (at 123.19 121.92 90)
       (effects (font (size 1.27 1.27)))
     )
@@
       (project "PLC 32 V2"
         (path "/d17a54f1-6eda-453f-95e1-42a53b02a1c3/e0987795-0f8d-4564-9094-c23cc01406e8"
-          (reference "R25") (unit 1) (value "220 ohm") (footprint "Resistor_SMD:R_0603_1608Metric")
+          (reference "R19") (unit 1) (value "220 ohm") (footprint "Resistor_SMD:R_0603_1608Metric")
         )
       )
@@
   (symbol (lib_id "Device:R") (at 118.11 140.97 90) (unit 1)
     (in_bom yes) (on_board yes) (dnp no)
-    (property "Reference" "R24" (at 115.57 144.78 90)
+    (property "Reference" "R18" (at 115.57 144.78 90)
       (effects (font (size 1.27 1.27)))
     )
@@
       (project "PLC 32 V2"
         (path "/d17a54f1-6eda-453f-95e1-42a53b02a1c3/e0987795-0f8d-4564-9094-c23cc01406e8"
-          (reference "R24") (unit 1) (value "220 ohm") (footprint "Resistor_SMD:R_0603_1608Metric")
+          (reference "R18") (unit 1) (value "220 ohm") (footprint "Resistor_SMD:R_0603_1608Metric")
         )
       )
@@
   (symbol (lib_id "Device:R") (at 118.11 132.08 90) (unit 1)
     (in_bom yes) (on_board yes) (dnp no)
-    (property "Reference" "R23" (at 115.57 129.54 90)
+    (property "Reference" "R17" (at 115.57 129.54 90)
       (effects (font (size 1.27 1.27)))
     )
@@
       (project "PLC 32 V2"
         (path "/d17a54f1-6eda-453f-95e1-42a53b02a1c3/e0987795-0f8d-4564-9094-c23cc01406e8"
-          (reference "R23") (unit 1) (value "220 ohm") (footprint "Resistor_SMD:R_0603_1608Metric")
+          (reference "R17") (unit 1) (value "220 ohm") (footprint "Resistor_SMD:R_0603_1608Metric")
         )
       )
@@
   (symbol (lib_id "Device:R") (at 76.2 132.08 90) (unit 1)
     (in_bom yes) (on_board yes) (dnp no) (fields_autoplaced)
-    (property "Reference" "R22" (at 76.2 125.73 90)
+    (property "Reference" "R16" (at 76.2 125.73 90)
       (effects (font (size 1.27 1.27)))
     )
@@
       (project "PLC 32 V2"
         (path "/d17a54f1-6eda-453f-95e1-42a53b02a1c3/e0987795-0f8d-4564-9094-c23cc01406e8"
-          (reference "R22") (unit 1) (value "220 ohm") (footprint "Resistor_SMD:R_0603_1608Metric_Pad0.98x0.95mm_HandSolder")
+          (reference "R16") (unit 1) (value "220 ohm") (footprint "Resistor_SMD:R_0603_1608Metric_Pad0.98x0.95mm_HandSolder")
         )
       )
@@
   (symbol (lib_id "Isolator:ILD74") (at 95.25 134.62 0) (unit 1)
     (in_bom yes) (on_board yes) (dnp no) (fields_autoplaced)
-    (property "Reference" "U9" (at 95.25 127 0)
+    (property "Reference" "U5" (at 95.25 127 0)
       (effects (font (size 1.27 1.27)))
     )
@@
       (project "PLC 32 V2"
         (path "/d17a54f1-6eda-453f-95e1-42a53b02a1c3/e0987795-0f8d-4564-9094-c23cc01406e8"
-          (reference "U9") (unit 1) (value "LD74-X009T") (footprint "Package_DIP:DIP-8_W8.89mm_SMDSocket_LongPads")
+          (reference "U5") (unit 1) (value "LD74-X009T") (footprint "Package_DIP:DIP-8_W8.89mm_SMDSocket_LongPads")
         )
       )
