File: salida4.kicad_sch (KiCad schematic)
At the start: 7 parts, among them Q5 FQP27P06, U9 LD74-X009T

Commit message: add
Parts:
- renumbered R26 to R20, R27 to R21, R28 to R22, R29 to R23, R30 to R24, U9 to U5
Changed lines of the file:
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@@
   (symbol (lib_id "Device:R") (at 123.19 127 90) (unit 1)
     (in_bom yes) (on_board yes) (dnp no)
-    (property "Reference" "R28" (at 120.65 125.73 90)
+    (property "Reference" "R22" (at 120.65 125.73 90)
       (effects (font (size 1.27 1.27)))
     )
@@
       (project "PLC 32 V2"
         (path "/d17a54f1-6eda-453f-95e1-42a53b02a1c3/d14d4c68-ec37-47aa-9929-a5e7ffbf99b8"
-          (reference "R28") (unit 1) (value "220 ohm") (footprint "Resistor_SMD:R_0603_1608Metric")
+          (reference "R22") (unit 1) (value "220 ohm") (footprint "Resistor_SMD:R_0603_1608Metric")
         )
       )
@@
   (symbol (lib_id "Device:R") (at 123.19 135.89 90) (unit 1)
     (in_bom yes) (on_board yes) (dnp no)
-    (property "Reference" "R29" (at 118.11 138.43 90)
+    (property "Reference" "R23" (at 118.11 138.43 90)
       (effects (font (size 1.27 1.27)))
     )
@@
       (project "PLC 32 V2"
         (path "/d17a54f1-6eda-453f-95e1-42a53b02a1c3/d14d4c68-ec37-47aa-9929-a5e7ffbf99b8"
-          (reference "R29") (unit 1) (value "220 ohm") (footprint "Resistor_SMD:R_0603_1608Metric")
+          (reference "R23") (unit 1) (value "220 ohm") (footprint "Resistor_SMD:R_0603_1608Metric")
         )
       )
@@
   (symbol (lib_id "Device:R") (at 81.28 127 90) (unit 1)
     (in_bom yes) (on_board yes) (dnp no) (fields_autoplaced)
-    (property "Reference" "R27" (at 81.28 120.65 90)
+    (property "Reference" "R21" (at 81.28 120.65 90)
       (effects (font (size 1.27 1.27)))
     )
@@
       (project "PLC 32 V2"
         (path "/d17a54f1-6eda-453f-95e1-42a53b02a1c3/d14d4c68-ec37-47aa-9929-a5e7ffbf99b8"
-          (reference "R27") (unit 1) (value "220 ohm") (footprint "Resistor_SMD:R_0603_1608Metric")
+          (reference "R21") (unit 1) (value "220 ohm") (footprint "Resistor_SMD:R_0603_1608Metric")
         )
       )
@@
   (symbol (lib_id "Device:R") (at 132.08 120.65 90) (unit 1)
     (in_bom yes) (on_board yes) (dnp no)
-    (property "Reference" "R30" (at 128.27 118.11 90)
+    (property "Reference" "R24" (at 128.27 118.11 90)
       (effects (font (size 1.27 1.27)))
     )
@@
       (project "PLC 32 V2"
         (path "/d17a54f1-6eda-453f-95e1-42a53b02a1c3/d14d4c68-ec37-47aa-9929-a5e7ffbf99b8"
-          (reference "R30") (unit 1) (value "220 ohm") (footprint "Resistor_SMD:R_0603_1608Metric")
+          (reference "R24") (unit 1) (value "220 ohm") (footprint "Resistor_SMD:R_0603_1608Metric")
         )
       )
@@
   (symbol (lib_id "Device:R") (at 71.12 134.62 0) (unit 1)
     (in_bom yes) (on_board yes) (dnp no) (fields_autoplaced)
-    (property "Reference" "R26" (at 73.66 133.3499 0)
+    (property "Reference" "R20" (at 73.66 133.3499 0)
       (effects (font (size 1.27 1.27)) (justify left))
     )
@@
       (project "PLC 32 V2"
         (path "/d17a54f1-6eda-453f-95e1-42a53b02a1c3/d14d4c68-ec37-47aa-9929-a5e7ffbf99b8"
-          (reference "R26") (unit 1) (value "10k") (footprint "Resistor_SMD:R_0603_1608Metric")
+          (reference "R20") (unit 1) (value "10k") (footprint "Resistor_SMD:R_0603_1608Metric")
         )
       )
@@
   (symbol (lib_id "Isolator:ILD74") (at 100.33 129.54 0) (unit 2)
     (in_bom yes) (on_board yes) (dnp no) (fields_autoplaced)
-    (property "Reference" "U9" (at 100.33 121.92 0)
+    (property "Reference" "U5" (at 100.33 121.92 0)
       (effects (font (size 1.27 1.27)))
     )
@@
       (project "PLC 32 V2"
         (path "/d17a54f1-6eda-453f-95e1-42a53b02a1c3/d14d4c68-ec37-47aa-9929-a5e7ffbf99b8"
-          (reference "U9") (unit 2) (value "LD74-X009T") (footprint "Package_DIP:DIP-8_W8.89mm_SMDSocket_LongPads")
-        )
-      )
+          (reference "U5") (unit 2) (value "LD74-X009T") (footprint "Package_DIP:DIP-8_W8.89mm_SMDSocket_LongPads")
+        )
+      )
