File: salida5.kicad_sch (KiCad schematic)
At the start: 7 parts, among them Q6 FQP27P06, U10 LD74-X009T

Commit message: add
Parts:
- renumbered R31 to R25, R32 to R26, R33 to R27, R34 to R28, R35 to R29, U10 to U6
Changed lines of the file:
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@@
   (symbol (lib_id "Device:R") (at 68.58 129.54 0) (unit 1)
     (in_bom yes) (on_board yes) (dnp no) (fields_autoplaced)
-    (property "Reference" "R31" (at 71.12 128.2699 0)
+    (property "Reference" "R25" (at 71.12 128.2699 0)
       (effects (font (size 1.27 1.27)) (justify left))
     )
@@
       (project "PLC 32 V2"
         (path "/d17a54f1-6eda-453f-95e1-42a53b02a1c3/64b407cd-5d00-473d-9ef6-2525490a4831"
-          (reference "R31") (unit 1) (value "10k") (footprint "Resistor_SMD:R_0603_1608Metric")
+          (reference "R25") (unit 1) (value "10k") (footprint "Resistor_SMD:R_0603_1608Metric")
         )
       )
@@
   (symbol (lib_id "Device:R") (at 120.65 130.81 90) (unit 1)
     (in_bom yes) (on_board yes) (dnp no)
-    (property "Reference" "R34" (at 124.46 134.62 90)
+    (property "Reference" "R28" (at 124.46 134.62 90)
       (effects (font (size 1.27 1.27)))
     )
@@
       (project "PLC 32 V2"
         (path "/d17a54f1-6eda-453f-95e1-42a53b02a1c3/64b407cd-5d00-473d-9ef6-2525490a4831"
-          (reference "R34") (unit 1) (value "220 ohm") (footprint "Resistor_SMD:R_0603_1608Metric")
+          (reference "R28") (unit 1) (value "220 ohm") (footprint "Resistor_SMD:R_0603_1608Metric")
         )
       )
@@
   (symbol (lib_id "Device:R") (at 129.54 115.57 90) (unit 1)
     (in_bom yes) (on_board yes) (dnp no)
-    (property "Reference" "R35" (at 127 111.76 90)
+    (property "Reference" "R29" (at 127 111.76 90)
       (effects (font (size 1.27 1.27)))
     )
@@
       (project "PLC 32 V2"
         (path "/d17a54f1-6eda-453f-95e1-42a53b02a1c3/64b407cd-5d00-473d-9ef6-2525490a4831"
-          (reference "R35") (unit 1) (value "220 ohm") (footprint "Resistor_SMD:R_0603_1608Metric")
+          (reference "R29") (unit 1) (value "220 ohm") (footprint "Resistor_SMD:R_0603_1608Metric")
         )
       )
@@
   (symbol (lib_id "Isolator:ILD74") (at 97.79 124.46 0) (unit 1)
     (in_bom yes) (on_board yes) (dnp no) (fields_autoplaced)
-    (property "Reference" "U10" (at 97.79 116.84 0)
+    (property "Reference" "U6" (at 97.79 116.84 0)
       (effects (font (size 1.27 1.27)))
     )
@@
       (project "PLC 32 V2"
         (path "/d17a54f1-6eda-453f-95e1-42a53b02a1c3/64b407cd-5d00-473d-9ef6-2525490a4831"
-          (reference "U10") (unit 1) (value "LD74-X009T") (footprint "Package_DIP:DIP-8_W8.89mm_SMDSocket_LongPads")
+          (reference "U6") (unit 1) (value "LD74-X009T") (footprint "Package_DIP:DIP-8_W8.89mm_SMDSocket_LongPads")
         )
       )
@@
   (symbol (lib_id "Device:R") (at 120.65 121.92 90) (unit 1)
     (in_bom yes) (on_board yes) (dnp no)
-    (property "Reference" "R33" (at 116.84 119.38 90)
+    (property "Reference" "R27" (at 116.84 119.38 90)
       (effects (font (size 1.27 1.27)))
     )
@@
       (project "PLC 32 V2"
         (path "/d17a54f1-6eda-453f-95e1-42a53b02a1c3/64b407cd-5d00-473d-9ef6-2525490a4831"
-          (reference "R33") (unit 1) (value "220 ohm") (footprint "Resistor_SMD:R_0603_1608Metric")
+          (reference "R27") (unit 1) (value "220 ohm") (footprint "Resistor_SMD:R_0603_1608Metric")
         )
       )
@@
   (symbol (lib_id "Device:R") (at 78.74 121.92 90) (unit 1)
     (in_bom yes) (on_board yes) (dnp no) (fields_autoplaced)
-    (property "Reference" "R32" (at 78.74 115.57 90)
+    (property "Reference" "R26" (at 78.74 115.57 90)
       (effects (font (size 1.27 1.27)))
     )
@@
       (project "PLC 32 V2"
         (path "/d17a54f1-6eda-453f-95e1-42a53b02a1c3/64b407cd-5d00-473d-9ef6-2525490a4831"
-          (reference "R32") (unit 1) (value "220 ohm") (footprint "Resistor_SMD:R_0603_1608Metric")
+          (reference "R26") (unit 1) (value "220 ohm") (footprint "Resistor_SMD:R_0603_1608Metric")
         )
       )
