File: salida6.kicad_sch (KiCad schematic)
At the start: 7 parts, among them Q7 FQP27P06, U10 LD74-X009T

Commit message: add
Parts:
- renumbered R36 to R30, R37 to R31, R38 to R32, R39 to R33, R40 to R34, U10 to U6
Changed lines of the file:
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@@
   (symbol (lib_id "Device:R") (at 80.01 127 90) (unit 1)
     (in_bom yes) (on_board yes) (dnp no)
-    (property "Reference" "R37" (at 74.93 124.46 90)
+    (property "Reference" "R31" (at 74.93 124.46 90)
       (effects (font (size 1.27 1.27)))
     )
@@
       (project "PLC 32 V2"
         (path "/d17a54f1-6eda-453f-95e1-42a53b02a1c3/4109c560-1e4d-481f-b3b5-bb77ed9700b9"
-          (reference "R37") (unit 1) (value "220 ohm") (footprint "Resistor_SMD:R_0603_1608Metric")
+          (reference "R31") (unit 1) (value "220 ohm") (footprint "Resistor_SMD:R_0603_1608Metric")
         )
       )
@@
   (symbol (lib_id "Isolator:ILD74") (at 99.06 129.54 0) (unit 2)
     (in_bom yes) (on_board yes) (dnp no) (fields_autoplaced)
-    (property "Reference" "U10" (at 99.06 121.92 0)
+    (property "Reference" "U6" (at 99.06 121.92 0)
       (effects (font (size 1.27 1.27)))
     )
@@
       (project "PLC 32 V2"
         (path "/d17a54f1-6eda-453f-95e1-42a53b02a1c3/4109c560-1e4d-481f-b3b5-bb77ed9700b9"
-          (reference "U10") (unit 2) (value "LD74-X009T") (footprint "Package_DIP:DIP-8_W8.89mm_SMDSocket_LongPads")
+          (reference "U6") (unit 2) (value "LD74-X009T") (footprint "Package_DIP:DIP-8_W8.89mm_SMDSocket_LongPads")
         )
       )
@@
   (symbol (lib_id "Device:R") (at 121.92 135.89 90) (unit 1)
     (in_bom yes) (on_board yes) (dnp no)
-    (property "Reference" "R39" (at 118.11 139.7 90)
+    (property "Reference" "R33" (at 118.11 139.7 90)
       (effects (font (size 1.27 1.27)))
     )
@@
       (project "PLC 32 V2"
         (path "/d17a54f1-6eda-453f-95e1-42a53b02a1c3/4109c560-1e4d-481f-b3b5-bb77ed9700b9"
-          (reference "R39") (unit 1) (value "220 ohm") (footprint "Resistor_SMD:R_0603_1608Metric")
+          (reference "R33") (unit 1) (value "220 ohm") (footprint "Resistor_SMD:R_0603_1608Metric")
         )
       )
@@
   (symbol (lib_id "Device:R") (at 121.92 127 90) (unit 1)
     (in_bom yes) (on_board yes) (dnp no)
-    (property "Reference" "R38" (at 118.11 124.46 90)
+    (property "Reference" "R32" (at 118.11 124.46 90)
       (effects (font (size 1.27 1.27)))
     )
@@
       (project "PLC 32 V2"
         (path "/d17a54f1-6eda-453f-95e1-42a53b02a1c3/4109c560-1e4d-481f-b3b5-bb77ed9700b9"
-          (reference "R38") (unit 1) (value "220 ohm") (footprint "Resistor_SMD:R_0603_1608Metric")
+          (reference "R32") (unit 1) (value "220 ohm") (footprint "Resistor_SMD:R_0603_1608Metric")
         )
       )
@@
   (symbol (lib_id "Device:R") (at 69.85 134.62 0) (unit 1)
     (in_bom yes) (on_board yes) (dnp no) (fields_autoplaced)
-    (property "Reference" "R36" (at 72.39 133.3499 0)
+    (property "Reference" "R30" (at 72.39 133.3499 0)
       (effects (font (size 1.27 1.27)) (justify left))
     )
@@
       (project "PLC 32 V2"
         (path "/d17a54f1-6eda-453f-95e1-42a53b02a1c3/4109c560-1e4d-481f-b3b5-bb77ed9700b9"
-          (reference "R36") (unit 1) (value "10k") (footprint "Resistor_SMD:R_0603_1608Metric")
+          (reference "R30") (unit 1) (value "10k") (footprint "Resistor_SMD:R_0603_1608Metric")
         )
       )
@@
   (symbol (lib_id "Device:R") (at 130.81 120.65 90) (unit 1)
     (in_bom yes) (on_board yes) (dnp no)
-    (property "Reference" "R40" (at 125.73 116.84 90)
+    (property "Reference" "R34" (at 125.73 116.84 90)
       (effects (font (size 1.27 1.27)))
     )
@@
       (project "PLC 32 V2"
         (path "/d17a54f1-6eda-453f-95e1-42a53b02a1c3/4109c560-1e4d-481f-b3b5-bb77ed9700b9"
-          (reference "R40") (unit 1) (value "220 ohm") (footprint "Resistor_SMD:R_0603_1608Metric")
+          (reference "R34") (unit 1) (value "220 ohm") (footprint "Resistor_SMD:R_0603_1608Metric")
         )
       )
